File: BumpyBoiTracky/BumpyBoiTracky.kicad_pcb (KiCad board)
At the start: 2 copper layers, 76 parts, among them J10 Conn_01x03_Female, J11 Conn_01x04_Female, J12 Conn_01x03_Female, J2 Conn_01x04_Female, J3 Conn_01x04_Female, J4 Conn_01x08_Female, J5 Conn_01x08_Female, J6 Conn_01x08_Female, J7 Conn_01x08_Female, J8 ICSP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

Commit message: Began layout for circuit board
Parts:
- added J1: USB_C_Receptacle, BumpyBoiTracky:Amphenol_USB-C_10164359-00011LF, F.Cu at (141.4, 73.1)
- moved R2 98.5 mm to (141.4, 75.5), turned to 180 degrees
- moved JP29 79.8 mm to (148.7, 116.7), turned to 90 degrees
- moved JP31 78.2 mm to (151.2, 116.7), turned to 90 degrees
- moved JP33 78.0 mm to (141.1, 110.3), turned to 180 degrees
- moved JP32 76.8 mm to (153.8, 116.7), turned to 90 degrees
- moved JP30 75.5 mm to (156.3, 116.7), turned to 90 degrees
- moved JP35 75.2 mm to (141.1, 107.8), turned to 180 degrees
- moved J9 75.0 mm to (148.7, 112.9), turned to 90 degrees
- moved JP36 72.4 mm to (141.1, 105.2), turned to 180 degrees
- moved J12 69.0 mm to (144.9, 105.3), turned to 0 degrees
- moved U2 66.2 mm to (152.5, 107.8), turned to 90 degrees
- moved JP38 66.0 mm to (148.7, 80.9), turned to 90 degrees
- moved J10 65.2 mm to (160.1, 110.3), turned to 180 degrees
- moved C5 64.2 mm to (155.7, 107.8), turned to 90 degrees
- moved R9 63.6 mm to (147.9, 83.4), turned to 0 degrees
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Routing:
- net +5V: track 0.00 -> 96.9 mm, vias 0 -> 11
- net /INT1: track 0.00 -> 91.0 mm, vias 0 -> 2
- net /INT2: track 0.00 -> 72.7 mm, vias 0 -> 2
- net Net-(J7-Pad5): track 0.00 -> 55.0 mm
- net Net-(J6-Pad1): track 0.00 -> 35.8 mm
- net /Controller/D0: track 0.00 -> 34.8 mm, vias 0 -> 1
- net /~{CS}: track 0.00 -> 32.0 mm, vias 0 -> 2
- net /MISO: track 0.00 -> 30.3 mm, vias 0 -> 2
- net Net-(J5-Pad8): track 0.00 -> 30.0 mm
- net Net-(C3-Pad1): track 0.00 -> 28.2 mm
- net Net-(C4-Pad1): track 0.00 -> 27.5 mm
- net Net-(J5-Pad7): track 0.00 -> 26.8 mm
- net /MOSI: track 0.00 -> 25.5 mm
- net GND: track 0.00 -> 21.9 mm, vias 0 -> 19
- net Net-(C2-Pad1): track 0.00 -> 17.2 mm
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- added copper zone on B.Cu, net +5V
- added copper zone on B.Cu, net GND
- added copper zone on F.Cu, net GND
Other:
- board outline added: 86 x 64.8 mm
