File: BumpyBoiTracky/converter.kicad_sch (KiCad schematic)
At the start: 11 parts, among them Q1 Q_PMOS_GSD, U3 LM3475

Commit message: Began layout for circuit board
Changed lines of the file:
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@@
+    (stroke (width 0) (type default) (color 0 0 0 0))
+  )
+  (wire (pts (xy 106.68 72.39) (xy 106.68 76.2))
     (stroke (width 0) (type default) (color 0 0 0 0))
   )
@@
     (effects (font (size 1.27 1.27)) (justify left))
   )
-  (hierarchical_label "+5V" (shape input) (at 115.57 76.2 90)
+  (hierarchical_label "+5V" (shape input) (at 106.68 72.39 0)
     (effects (font (size 1.27 1.27)) (justify left))
   )
